Commit message: bugfix

File: high_dof_description/urdf/antro3.xacro (robot description, xacro)
@@ -72,5 +72,5 @@
     <origin xyz="0 ${-upper_arm_length/2} 0" rpy="1.5708 0 0" />
     <geometry>
-      <cylinder length="${-upper_arm_length}"
+      <cylinder length="${upper_arm_length}"
       radius="${upper_arm_radius}" />
     </geometry>
